File: hardware/kicad/IMpack.kicad_sch (KiCad schematic)
At the start: 0 parts

Commit message: added board production files
Other:
- title: STM32 Accelerometer -> IMpack
Changed lines of the file:
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@@
 	(paper "A")
 	(title_block
-		(title "STM32 Accelerometer")
+		(title "IMpack")
 		(date "2023-12-14")
 		(rev "1.0")
